Commit message: Final Xacro

File: src/robot_description/urdf/Robot.urdf.xacro (robot description, xacro)
@@ -1,84 +1,5 @@
 <?xml version="1.0"?>
 <robot name="Robot" xmlns:xacro="http://www.ros.org/wiki/xacro">
-    <!-- ========================== -->
-    <!--            Variables       -->
-    <!-- ========================== -->
-    <xacro:property name="base_length" value="0.6"/>
-    <xacro:property name="base_width" value="0.4"/>
-    <xacro:property name="base_height" value="0.2"/>
-    <xacro:property name="wheel_radius" value="0.1"/>
-    <xacro:property name="wheel_length" value="0.05"/>
-    <!-- ====================================================================================== -->
-    <!-- ========================== -->
-    <!--   Create Macros (Functions)-->
-    <!-- ========================== -->
-    <xacro:macro name="wheel_link" params="prefix">
-        <link name="${prefix}_wheel">
-            <visual>
-                <geometry>
-                    <cylinder radius="${wheel_radius}" length="${wheel_length}"/>
-                </geometry>
-                <origin xyz="0.0 0.0 0.0" rpy="${pi/2} 0.0 0.0"/>
-                <material name="Blue"/>
-            </visual>
-        </link>
-    </xacro:macro>
-    <!-- ====================================================================================== -->
-    <!-- ========================== -->
-    <!--            LINKS           -->
-    <!-- ========================== -->
-    <xacro:wheel_link prefix="right"/>
-    <xacro:wheel_link prefix="left"/>
-    <material name="Green">
-        <color rgba="0.4 0.5 0.0 1"/>
-    </material>
-    <material name="Blue">
-        <color rgba="0.0 0.5 0.0 1"/>
-    </material>
-    <link name="base_link">
-        <visual>
-            <geometry>
-                <box size="${base_length} ${base_width} ${base_height}"/>
-            </geometry>
-            <origin xyz="0 0 ${base_height / 2}" rpy="0 0 0"/>
-            <material name="Green"/>
-        </visual>
-    </link>
-    <link name="Caster_wheel">
-        <visual>
-            <geometry>
-                <sphere radius="0.05"/>
-            </geometry>
-            <origin xyz="0.0 0.0 0.0" rpy="0.0 0.0 0.0"/>
-        </visual>
-    </link>
-    <link name="base_footprint"/>
-    <!-- ====================================================================================== -->
-    <!-- ========================== -->
-    <!--            JOINTS          -->
-    <!-- ========================== -->
-    <joint name="right_wheel_Joint" type="revolute">
-        <origin xyz="-0.15 -0.225 0.0" rpy="0.0 0.0 0.0"/>
-        <parent link="base_link"/>
-        <child link="right_wheel"/>
-        <axis xyz="0.0 1.0 0.0"/>
-        <limit lower="-3.14" upper="3.14" effort="100" velocity="100"/>
-    </joint>
-    <joint name="left_wheel_Joint" type="revolute">
-        <origin xyz="-0.15 0.225 0.0" rpy="0.0 0.0 0.0"/>
-        <parent link="base_link"/>
-        <child link="left_wheel"/>
-        <axis xyz="0.0 -1.0 0.0"/>
-        <limit lower="-3.14" upper="3.14" effort="100" velocity="100"/>
-    </joint>
-    <joint name="base_caster_wheel_joint" type="fixed">
-        <origin xyz="0.2 0.0 -0.05"/>
-        <parent link="base_link"/>
-        <child link="Caster_wheel"/>
-    </joint>
-    <joint name="base_joint" type="fixed">
-        <origin xyz="0.0 0.0 -0.1" rpy="0.0 0.0 0.0"/>
-        <parent link="base_link"/>
-        <child link="base_footprint"/>
-    </joint>
+    <xacro:include filename="Common_proprties.xacro"/>
+    <xacro:include filename="mobile_base.xacro"/>
 </robot>
