Commit message: Add collisons and Inertia

File: src/robot_description/urdf/Common_proprties.xacro (robot description, xacro)
@@ -7,3 +7,33 @@
         <color rgba="0.0 0.5 0.0 1"/>
     </material>
+<!--BOX INERTIA MACRO-->
+    <xacro:macro name="box_inertia" params="m l w h xyz rpy">
+        <inertial>
+            <origin xyz="${xyz}" rpy="${rpy}"/>
+            <mass value="${m}"/>
+            <inertia ixx="${(m/12) * (h*h + l+l)}" ixy="0.0" ixz="0.0"
+                     iyy="${(m/12) * (w*w + l+l)}" iyz="0.0"
+                     izz="${(m/12) * (w*w + h+h)}"/>
+        </inertial>
+    </xacro:macro>
+<!--WHEEL INERTIA MACRO-->
+    <xacro:macro name="cylinder_inerta" params="m r h xyz rpy">
+        <inertial>
+            <origin xyz="${xyz}" rpy="${rpy}"/>
+            <mass value="${m}"/>
+            <inertia ixx="${(m/12) * (3*r*r)+(h*h)}" ixy="0.0" ixz="0.0"
+                     iyy="${(m/12) * (3*r*r)+(h*h)}" iyz="0.0"
+                     izz="${(m/2)  *  ( r * r )}"/>
+        </inertial>
+    </xacro:macro>
+<!--BALL INERTIA MACRO-->
+    <xacro:macro name="ball_inertia" params= " m r xyz rpy">
+        <inertial>
+            <origin xyz="${xyz}" rpy="${rpy}"/>
+            <mass value="${m}"/>
+            <inertia ixx="${(2/5) * m *r *r }" ixy="0.0" ixz="0.0"
+                     iyy="${(2/5) * m *r *r }" iyz="0.0"
+                     izz="${(2/5) * m *r *r }"/>
+        </inertial>
+    </xacro:macro>
 </robot>

File: src/robot_description/urdf/mobile_base.xacro (robot description, xacro)
@@ -22,4 +22,11 @@
                 <material name="Blue"/>
             </visual>
+            <collision>
+                <geometry>
+                    <cylinder radius="${wheel_radius}" length="${wheel_length}"/>
+                </geometry>
+                <origin xyz="0.0 0.0 0.0" rpy="${pi/2} 0.0 0.0"/>
+            </collision>
+            <xacro:cylinder_inerta m="1.0" r="${wheel_radius}" h="${wheel_length}" xyz="0.0 0.0 0.0" rpy="${pi/2} 0.0 0.0"/>
         </link>
     </xacro:macro>
@@ -38,4 +45,11 @@
             <material name="Green"/>
         </visual>
+        <collision>
+            <geometry>
+                <box size="${base_length} ${base_width} ${base_height}"/>
+            </geometry>
+            <origin xyz="0 0 ${base_height / 2}" rpy="0 0 0"/>
+        </collision>
+        <xacro:box_inertia m="5.0" l="${base_length}" w="${base_width}" h="${base_height}"  xyz="0.0 0.0 0.0" rpy="0.0 0.0 0.0"/>
     </link>
     <link name="Caster_wheel">
@@ -46,4 +60,11 @@
             <origin xyz="0.0 0.0 0.0" rpy="0.0 0.0 0.0"/>
         </visual>
+        <collision>
+            <geometry>
+                <sphere radius="0.05"/>
+            </geometry>
+            <origin xyz="0.0 0.0 0.0" rpy="0.0 0.0 0.0"/>
+        </collision>
+        <xacro:ball_inertia m="0.1" r="0.05" xyz="0.0 0.0 0.0" rpy="0.0 0.0 0.0"/>
     </link>
     <link name="base_footprint"/>

Commit message: create launch file for Gazebo

File: src/robot_description/urdf/Common_proprties.xacro (robot description, xacro)
@@ -18,11 +18,11 @@
     </xacro:macro>
 <!--WHEEL INERTIA MACRO-->
-    <xacro:macro name="cylinder_inerta" params="m r h xyz rpy">
+    <xacro:macro name="cylinder_inertia" params="m r h xyz rpy">
         <inertial>
             <origin xyz="${xyz}" rpy="${rpy}"/>
             <mass value="${m}"/>
             <inertia ixx="${(m/12) * (3*r*r)+(h*h)}" ixy="0.0" ixz="0.0"
-                     iyy="${(m/12) * (3*r*r)+(h*h)}" iyz="0.0"
-                     izz="${(m/2)  *  ( r * r )}"/>
+                    iyy="${(m/12) * (3*r*r)+(h*h)}" iyz="0.0"
+                    izz="${(m/12) * (3*r*r + h*h)}"/>
         </inertial>
     </xacro:macro>

File: src/robot_description/urdf/mobile_base.xacro (robot description, xacro)
@@ -28,5 +28,5 @@
                 <origin xyz="0.0 0.0 0.0" rpy="${pi/2} 0.0 0.0"/>
             </collision>
-            <xacro:cylinder_inerta m="1.0" r="${wheel_radius}" h="${wheel_length}" xyz="0.0 0.0 0.0" rpy="${pi/2} 0.0 0.0"/>
+            <xacro:cylinder_inertia m="1.0" r="${wheel_radius}" h="${wheel_length}" xyz="0.0 0.0 0.0" rpy="${pi/2} 0.0 0.0"/>
         </link>
     </xacro:macro>
